File: 6key.sch (KiCad schematic (older format))
At the start: 17 parts

Commit message: finished-ish schematic
Parts:
- added D1, D2, D3, D4, D5, D6: D_Small, Diode_SMD:D_SOD-123, symbol Device:D_Small
- added SW2: SW_Push, random-keyboard-parts:SKQG-1155865, symbol Switch:SW_Push
- added U2: ProMicro, footprint:ARDUINO_PRO_MICRO, symbol promicro:ProMicro
- C1, C2, C3: renamed from C?; footprint (none) -> Capacitor_SMD:C_0805_2012Metric_Pad1.15x1.40mm_HandSolder
- F1: renamed from F?; footprint (none) -> Fuse:Fuse_1206_3216Metric_Pad1.42x1.75mm_HandSolder
- J1: renamed from J?; footprint (none) -> random-keyboard-parts:Molex-0548190519
- MX1, MX2, MX3, MX4, MX5, MX6: renamed from MX?; footprint (none) -> MX_Only:MXOnly-1U-NoLED
- R1: renamed from R?; footprint (none) -> Resistor_SMD:R_0815_2038Metric_Pad1.53x4.00mm_HandSolder
- R2, R3: renamed from R?; footprint (none) -> Resistor_SMD:R_0805_2012Metric_Pad1.15x1.40mm_HandSolder
- SW1: renamed from SW?; footprint (none) -> random-keyboard-parts:SKQG-1155865
- Y1: renamed from Y?; footprint (none) -> Crystal:Crystal_SMD_3225-4Pin_3.2x2.5mm_HandSoldering
- gave numbers to parts that had none: 1
Connections:
- net labels added: COL0, COL1, COL2, ROW0, ROW1
- wire segments 42 -> 55
Other:
- moved on the sheet: MX2, MX4, MX6
